File: hw/Femtosat/USB.sch (KiCad schematic (older format))
At the start: 5 parts, among them J1 USB_B_Micro

Commit message: Added library for certain components. Symbols and footprints were associated.
Parts:
- C6: footprint Capacitor_SMD:C_0805_2012Metric_Pad1.15x1.40mm_HandSolder -> Capacitor_SMD:C_0603_1608Metric_Pad1.05x0.95mm_HandSolder
Changed lines of the file:
@@
 F 0 "C6" H 7615 4346 50  0000 L CNN
 F 1 "4.7nF" H 7615 4255 50  0000 L CNN
-F 2 "Capacitor_SMD:C_0805_2012Metric_Pad1.15x1.40mm_HandSolder" H 7538 4150 50  0001 C CNN
+F 2 "Capacitor_SMD:C_0603_1608Metric_Pad1.05x0.95mm_HandSolder" H 7538 4150 50  0001 C CNN
 F 3 "~" H 7500 4300 50  0001 C CNN
 	1    7500 4300

Commit message: Associated the new symbols to their respective footprints.
Parts:
- R2: footprint Resistor_SMD:R_0805_2012Metric_Pad1.15x1.40mm_HandSolder -> Resistor_SMD:R_0603_1608Metric
Changed lines of the file:
@@
 F 0 "R2" H 7970 4346 50  0000 L CNN
 F 1 "1M" H 7970 4255 50  0000 L CNN
-F 2 "Resistor_SMD:R_0805_2012Metric_Pad1.15x1.40mm_HandSolder" V 7830 4300 50  0001 C CNN
+F 2 "Resistor_SMD:R_0603_1608Metric" V 7830 4300 50  0001 C CNN
 F 3 "~" H 7900 4300 50  0001 C CNN
 	1    7900 4300
