File: hw/Femtosat/programmer.sch (KiCad schematic (older format))
At the start: 2 parts, among them J2 Programmer

Commit message: Associated the new symbols to their respective footprints.
Parts:
- J2: footprint (none) -> Connector_PinHeader_2.54mm:PinHeader_1x04_P2.54mm_Vertical
- R1: footprint (none) -> Resistor_SMD:R_0603_1608Metric_Pad1.05x0.95mm_HandSolder
Changed lines of the file:
@@
 F 0 "J2" H 4722 2982 50  0000 R CNN
 F 1 "Programmer" H 4722 3073 50  0000 R CNN
-F 2 "" H 4750 3100 50  0001 C CNN
+F 2 "Connector_PinHeader_2.54mm:PinHeader_1x04_P2.54mm_Vertical" H 4750 3100 50  0001 C CNN
 F 3 "~" H 4750 3100 50  0001 C CNN
 	1    4750 3100
@@
 U 1 1 5BFFC4E5
 P 4450 2700
-F 0 "R1" V 4657 2700 50  0000 C CNN
-F 1 "1k" V 4566 2700 50  0000 C CNN
-F 2 "" V 4380 2700 50  0001 C CNN
+F 0 "R1" V 4550 2700 50  0000 C CNN
+F 1 "1k" V 4450 2700 50  0000 C CNN
+F 2 "Resistor_SMD:R_0603_1608Metric_Pad1.05x0.95mm_HandSolder" V 4380 2700 50  0001 C CNN
 F 3 "~" H 4450 2700 50  0001 C CNN
 	1    4450 2700
