File: hw/Femtosat/communication.sch (KiCad schematic (older format))
At the start: 2 parts, among them J3 SMA, U4 RFM69HCW

Commit message: Added library for certain components. Symbols and footprints were associated.
Parts:
- J3: footprint (none) -> Antenna:SMA
- U4: footprint (none) -> Transceptor:RFM69HCW
Changed lines of the file:
@@
 F 0 "U4" H 5250 4000 50  0000 C CNN
 F 1 "RFM69HCW" H 5800 4000 50  0000 C CNN
-F 2 "" H 2300 5200 50  0001 C CNN
+F 2 "Transceptor:RFM69HCW" H 2300 5200 50  0001 C CNN
 F 3 "http://www.hoperf.com/upload/rf/RFM69HCW-V1.1.pdf" H 2300 5200 50  0001 C CNN
 	1    5600 3550
@@
 F 0 "J3" H 6800 3225 50  0000 L CNN
 F 1 "SMA" H 6800 3134 50  0000 L CNN
-F 2 "" H 6700 3250 50  0001 C CNN
+F 2 "Antenna:SMA" H 6700 3250 50  0001 C CNN
 F 3 "" H 6700 3250 50  0001 C CNN
 	1    6700 3250

Commit message: Added capacitors for the communication system.
Parts:
- added Ca7, Cb7: C, Capacitor_SMD:C_0603_1608Metric_Pad1.05x0.95mm_HandSolder, symbol Device:C
Connections:
- net 3.3V: now also Ca7.2, Cb7.2
- net GND: now also Ca7.1, Cb7.1
Changed lines of the file:
@@
 Wire Wire Line
 	5600 3050 5600 2950
-Wire Wire Line
-	5600 2950 5750 2950
 Text Label 5750 2950 2    50   ~ 0
 3.3V
@@
 Wire Wire Line
 	6700 3450 6700 3500
+$Comp
+L Device:C Ca7
+U 1 1 5BD8FE47
+P 6250 2850
+F 0 "Ca7" V 6150 2850 50  0000 C CNN
+F 1 "C" V 6250 2850 50  0000 C CNN
+F 2 "Capacitor_SMD:C_0603_1608Metric_Pad1.05x0.95mm_HandSolder" H 6288 2700 50  0001 C CNN
+F 3 "~" H 6250 2850 50  0001 C CNN
+	1    6250 2850
+	0    1    1    0
+$EndComp
+$Comp
+L Device:C Cb7
+U 1 1 5BD90136
+P 6250 3100
+F 0 "Cb7" V 6150 3100 50  0000 C CNN
+F 1 "C" V 6250 3100 50  0000 C CNN
+F 2 "Capacitor_SMD:C_0603_1608Metric_Pad1.05x0.95mm_HandSolder" H 6288 2950 50  0001 C CNN
+F 3 "~" H 6250 3100 50  0001 C CNN
+	1    6250 3100
+	0    1    1    0
+$EndComp
+Wire Wire Line
+	6100 2850 6050 2850
+Wire Wire Line
+	6050 2850 6050 2950
+Wire Wire Line
+	6050 3100 6100 3100
+Wire Wire Line
+	5600 2950 6050 2950
+Connection ~ 6050 2950
+Wire Wire Line
+	6050 2950 6050 3100
+Wire Wire Line
+	6400 2850 6450 2850
+Wire Wire Line
+	6450 2850 6450 3100
+Wire Wire Line
+	6450 3100 6400 3100
+Text Label 6450 2950 0    50   ~ 0
+GND
 $EndSCHEMATC

Commit message: Minor changes.
Connections:
- net ANT: now reaches J3.1 (In), U4.9 (ANT)
Changed lines of the file:
@@
 Text Label 6450 2950 0    50   ~ 0
 GND
+Text Label 6300 3250 2    50   ~ 0
+ANT
 $EndSCHEMATC
