File: hw/Femtosat/Femtosat.kicad_pcb (KiCad board)
At the start: 2 copper layers, 28 parts, among them J1 USB_B_Micro, J2 Programmer, J3 SMA, U0 AP7215-33YG-13, U2 TRH-G2, U3 XA1110, U4 RFM69HCW, Y1 32.768kHz

Commit message: Deleted the GPS device (moved to another PCB). Added the deploy-sensor (an interrupter). Moved the programmer to its own hierarchical sheet.
Parts:
- removed U3: XA1110, GPS:XA1110
- J2: footprint Connector_PinSocket_2.54mm:PinSocket_1x03_P2.54mm_Vertical -> Connector_PinHeader_2.54mm:PinHeader_1x04_P2.54mm_Vertical
- moved Y1 3.47 mm to (141.3, 64.5)
- moved Cc1 3.45 mm to (144.2, 62.9)
- moved Cc2 3.29 mm to (144.2, 66.1)
- moved J2 1.52 mm to (137.2, 54.6)
- renumbered Ue to U1
Connections:
- J2 pad 1: /SWDIO -> GND
- J2 pad 2: /SWCLK -> /RESET
- J2 pad 3: /RESET -> /SWCLK

Commit message: Associated the new symbols to their respective footprints.
Parts:
- removed R2: 1M, Resistor_SMD:R_0805_2012Metric_Pad1.15x1.40mm_HandSolder
Changed lines of the file:
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@@
     (tracks 0)
     (zones 0)
-    (modules 27)
+    (modules 26)
     (nets 61)
   )
@@
     (model ${KISYS3DMOD}/Resistor_SMD.3dshapes/R_0805_2012Metric.wrl
       (at (xyz 0 0 0))
-      (scale (xyz 1 1 1))
-      (rotate (xyz 0 0 0))
-    )
-  )
-  (module Resistor_SMD:R_0805_2012Metric_Pad1.15x1.40mm_HandSolder (layer F.Cu)
-    (at 118.6 67.3)
-    (descr "Resistor SMD 0805 (2012 Metric), square (rectangular) end terminal, IPC_7351 nominal with elongated pad for handsoldering. (Body size source: https://docs.google.com/spreadsheets/d/1BsfQQcO9C6DZCsRaXUlFlo91Tg2WpOkGARC1WS5S8t0/edit?usp=sharing), generated with kicad-footprint-generator")
-    (tags "resistor handsolder")
-    (attr smd)
-    (fp_text reference R2 (at 0 1.6) (layer F.SilkS)
-      (effects (font (size 1 1) (thickness 0.15)))
-    )
-    (fp_text value 1M (at 0 1.65) (layer F.Fab) hide
-      (effects (font (size 1 1) (thickness 0.15)))
-    )
-    (fp_text user %R (at 0 0) (layer F.Fab) hide
-      (effects (font (size 0.5 0.5) (thickness 0.08)))
-    )
-    (fp_line (start 1.85 0.95) (end -1.85 0.95) (layer F.CrtYd) (width 0.05))
-    (fp_line (start 1.85 -0.95) (end 1.85 0.95) (layer F.CrtYd) (width 0.05))
-    (fp_line (start -1.85 -0.95) (end 1.85 -0.95) (layer F.CrtYd) (width 0.05))
-    (fp_line (start -1.85 0.95) (end -1.85 -0.95) (layer F.CrtYd) (width 0.05))
-    (fp_line (start -0.261252 0.71) (end 0.261252 0.71) (layer F.SilkS) (width 0.12))
-    (fp_line (start -0.261252 -0.71) (end 0.261252 -0.71) (layer F.SilkS) (width 0.12))
-    (fp_line (start 1 0.6) (end -1 0.6) (layer F.Fab) (width 0.1))
-    (fp_line (start 1 -0.6) (end 1 0.6) (layer F.Fab) (width 0.1))
-    (fp_line (start -1 -0.6) (end 1 -0.6) (layer F.Fab) (width 0.1))
-    (fp_line (start -1 0.6) (end -1 -0.6) (layer F.Fab) (width 0.1))
-    (pad 2 smd roundrect (at 1.025 0) (size 1.15 1.4) (layers F.Cu F.Paste F.Mask) (roundrect_rratio 0.217391)
-      (net 2 GND))
-    (pad 1 smd roundrect (at -1.025 0) (size 1.15 1.4) (layers F.Cu F.Paste F.Mask) (roundrect_rratio 0.217391)
-      (net 4 "Net-(C6-Pad1)"))
-    (model ${KISYS3DMOD}/Resistor_SMD.3dshapes/R_0805_2012Metric.wrl
-      (at (xyz 0 0 0))

Commit message: Minor changes.
Parts:
- added J4: Battery, Connector_JST:JST_PH_S2B-PH-K_1x02_P2.00mm_Horizontal, F.Cu at (110.2, 78.8)
- added R2: 1M, Resistor_SMD:R_0603_1608Metric, F.Cu at (116.0, 60.5)
- added R3: 1k, Resistor_SMD:R_0603_1608Metric, F.Cu at (109.7, 71.8)
- added U3: AV4524, Interrupt:AV4524, F.Cu at (106.5, 71.8)
- C5, Ca7, Cb7, Cr1, Cr2, D3, J1, J3, U0, U4: moved to B.Cu
- JP1: value Jumper_NC_Dual -> POW_SEL
- R1: footprint Resistor_SMD:R_0805_2012Metric_Pad1.15x1.40mm_HandSolder -> Resistor_SMD:R_0603_1608Metric_Pad1.05x0.95mm_HandSolder
- moved Cb7 52.0 mm to (159.8, 60.3)
- moved Ca7 51.2 mm to (159.8, 58.8)
- moved Cr2 47.4 mm to (127.1, 80.1)
- moved U4 47.1 mm to (160.6, 71.5), turned to 90 degrees
- moved Cr1 44.0 mm to (127.1, 78.6)
- moved U0 43.3 mm to (121.9, 78.6), turned to 180 degrees
- moved C3b1 40.6 mm to (126.8, 60.3), turned to 270 degrees
- moved J3 39.9 mm to (153.6, 57.0), turned to 270 degrees
- moved JP1 32.4 mm to (123.9, 72.5), turned to 270 degrees
- moved J2 27.2 mm to (110.0, 55.5), turned to 90 degrees
- moved C3a1 25.3 mm to (134.0, 70.2), turned to 180 degrees
- moved C4 20.1 mm to (134.0, 71.8), turned to 180 degrees
- moved D3 17.0 mm to (126.5, 65.9)
- moved C5 8.23 mm to (132.1, 56.8)
- moved C6 7.65 mm to (113.3, 59.6), turned to 180 degrees
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Connections:
- net Net-(J3-Pad1) renamed /Communication/ANT
- Cr1 pad 1: /5V0 -> /VBUS
- Cr2 pad 1: /3V3 -> /Power/REG_OUT
- JP1 pad 1: /VBUS -> /Power/REG_OUT
- JP1 pad 2: /5V0 -> /3V3
- JP1 pad 3: /VIN -> /VBAT
- U0 pad 2: /5V0 -> /VBUS
- U0 pad 3: /3V3 -> /Power/REG_OUT
- U2 pad 1: /5V0 -> /3V3
- U2 pad 12: Net-(U2-Pad12) -> /SCL
- U2 pad 2: /5V0 -> /3V3
- U2 pad 9: Net-(U2-Pad9) -> /SDA
Routing:
- added copper zone on B.Cu, net GND
- added copper zone on F.Cu, net GND
Other:
- board outline added: 83.8 x 34 mm

Commit message: Routed all tracks.
Parts:
- removed JP1: POW_SEL, Connector_PinHeader_2.54mm:PinHeader_1x03_P2.54mm_Vertical
- removed R3: 1k, Resistor_SMD:R_0603_1608Metric
- added U5: XA1110, GPS:XA1110_I2C, F.Cu at (140.0, 69.0)
- Ca7, Cb7, U4: moved to F.Cu
- moved J3 16.7 mm to (170.0, 60.0)
- moved Cr2 12.8 mm to (114.3, 79.5), turned to 270 degrees
- moved Cr1 11.3 mm to (115.8, 79.5), turned to 270 degrees
- moved U0 7.50 mm to (115.8, 74.3), turned to 90 degrees
- moved L1 6.08 mm to (136.0, 70.5)
- moved C2a1 5.95 mm to (136.8, 66.5)
- moved C2b1 5.94 mm to (136.8, 68.0)
- moved U4 5.48 mm to (156.0, 68.5)
- moved C5 5.31 mm to (127.1, 58.5)
- moved R1 5.31 mm to (130.4, 58.5)
- moved Cc1 5.22 mm to (139.3, 61.2)
- moved Cc2 5.22 mm to (139.3, 64.5)
- moved Y1 5.22 mm to (136.4, 62.9)
- moved D3 5.21 mm to (121.5, 67.2)
- moved U1 5.16 mm to (128.5, 65.4)
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Connections:
- net /GPS_RST renamed Net-(U2-Pad7)
- Cr2 pad 1: /Power/REG_OUT -> /Power/REG_USB
- U0 pad 3: /Power/REG_OUT -> /Power/REG_USB
- U1 pad 29: /PIN_6 -> /TRX_RST
- U1 pad 30: /PIN_7 -> /TRX_NSS
- U1 pad 31: /PIN_0 -> /TRX_INT
- U2 pad : (no net) -> GND
- U2 pad 12: /SCL -> Net-(U2-Pad12)
- U2 pad 9: /SDA -> Net-(U2-Pad9)
- U3 pad 1: GND -> /3V3
- U3 pad 2: /DPL_STA -> /Power/REG_USB
- U3 pad 3: Net-(U3-Pad3) -> /VBAT
Routing:
- net /3V3: track 0.00 -> 143.3 mm, vias 0 -> 10
- net GND: track 0.00 -> 131.7 mm, vias 0 -> 24
- net /RX: track 0.00 -> 68.4 mm, vias 0 -> 2
- net /TX: track 0.00 -> 61.8 mm, vias 0 -> 2
- net /TRX_NSS: track 0.00 -> 45.2 mm, vias 0 -> 1
- net /TRX_RST: track 0.00 -> 41.0 mm, vias 0 -> 1
- net /MISO: track 0.00 -> 39.6 mm, vias 0 -> 1
- net /SCK: track 0.00 -> 37.9 mm, vias 0 -> 3
- net /TRX_INT: track 0.00 -> 36.1 mm, vias 0 -> 1
- net /MOSI: track 0.00 -> 33.7 mm, vias 0 -> 3
- net /VBUS: track 0.00 -> 22.6 mm, vias 0 -> 1
- net /SWCLK: track 0.00 -> 22.5 mm
- net /USB_P: track 0.00 -> 22.0 mm, vias 0 -> 1
- net /USB_N: track 0.00 -> 22.0 mm, vias 0 -> 1
- net /SCL: track 0.00 -> 20.1 mm, vias 0 -> 1
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Other:
- net class Default: via_dia 0.8 -> 1
- net class Power added: clearance 0.2, trace_width 0.5, via_dia 1, via_drill 0.4
- net class uC: via_drill 0.7 -> 0.4
