File: hw/PCB/USB.sch (KiCad schematic (older format))
At the start: 5 parts, among them J1 USB_B_Micro

Commit message: Added a footprint library for a micro SD card. Updated the schematic. Replaced the SAMD21G with the SAMD21E (32 pin variant). Added a data logger and a reset button.
Parts:
- removed D3: D_Schottky, Diode_SMD:D_SOD-523, symbol Device:D_Schottky
- added R4: 330, Resistor_SMD:R_0603_1608Metric, symbol Device:R
- renumbered C6 to C5, R2 to R3
Connections:
- net GND: no longer J1.6 (Shield)
- net ID: now also R4.2
- net USB_ID: now also R4.1
- net SHIELD: now reaches C5.1, D1.1 (GND), R3.1
- net SHIELD: now also J1.6 (Shield)
- net VBUS renamed VUSB
Other:
- moved on the sheet: C5, R3
Changed lines of the file:
@@
 $Descr A4 11693 8268
 encoding utf-8
-Sheet 3 5
+Sheet 3 6
 Title ""
 Date ""
@@
 $EndComp
 Text Label 5900 3150 2    50   ~ 0
-VBUS
+VUSB
 Text Label 5900 3350 2    50   ~ 0
 USB_DP
@@
 Text Label 6600 3550 2    50   ~ 0
 USB_ID
-Text Label 5200 3800 2    50   ~ 0
+Text Label 5300 3800 0    50   ~ 0
 GND
-Wire Wire Line
-	5200 3750 5200 3800
-Wire Wire Line
-	5200 3800 5250 3800
-Wire Wire Line
-	5300 3800 5300 3750
-Wire Wire Line
-	5250 3800 5250 3850
-Connection ~ 5250 3800
-Wire Wire Line
-	5250 3800 5300 3800
 $Comp
 L power:GND #PWR0102
 U 1 1 5B62BD38
-P 5250 3850
-F 0 "#PWR0102" H 5250 3600 50  0001 C CNN
-F 1 "GND" H 5255 3677 50  0000 C CNN
-F 2 "" H 5250 3850 50  0001 C CNN
-F 3 "" H 5250 3850 50  0001 C CNN
-	1    5250 3850
+P 5300 3850
+F 0 "#PWR0102" H 5300 3600 50  0001 C CNN
+F 1 "GND" H 5305 3677 50  0000 C CNN
+F 2 "" H 5300 3850 50  0001 C CNN
+F 3 "" H 5300 3850 50  0001 C CNN
+	1    5300 3850
 	1    0    0    -1
 $EndComp
@@
 $EndComp
 $Comp
-L Device:R R2
+L Device:R R3
 U 1 1 5B62BE0D
-P 7900 4300
-F 0 "R2" H 7970 4346 50  0000 L CNN
-F 1 "1M" H 7970 4255 50  0000 L CNN
-F 2 "Resistor_SMD:R_0603_1608Metric" V 7830 4300 50  0001 C CNN
-F 3 "~" H 7900 4300 50  0001 C CNN
-	1    7900 4300
+P 6750 4300
+F 0 "R3" H 6820 4346 50  0000 L CNN
+F 1 "1M" H 6820 4255 50  0000 L CNN
+F 2 "Resistor_SMD:R_0603_1608Metric" V 6680 4300 50  0001 C CNN
+F 3 "~" H 6750 4300 50  0001 C CNN
+	1    6750 4300
 	1    0    0    -1
 $EndComp
 $Comp
-L Device:C C6
+L Device:C C5
 U 1 1 5B62BE71
-P 7500 4300
-F 0 "C6" H 7615 4346 50  0000 L CNN
-F 1 "4.7nF" H 7615 4255 50  0000 L CNN
-F 2 "Capacitor_SMD:C_0603_1608Metric_Pad1.05x0.95mm_HandSolder" H 7538 4150 50  0001 C CNN
-F 3 "~" H 7500 4300 50  0001 C CNN
-	1    7500 4300
+P 6350 4300
+F 0 "C5" H 6465 4346 50  0000 L CNN
+F 1 "4.7nF" H 6465 4255 50  0000 L CNN
+F 2 "Capacitor_SMD:C_0603_1608Metric_Pad1.05x0.95mm_HandSolder" H 6388 4150 50  0001 C CNN
+F 3 "~" H 6350 4300 50  0001 C CNN
+	1    6350 4300
 	1    0    0    -1
 $EndComp
 Wire Wire Line
-	7500 4150 7500 4100
+	6350 4150 6350 4100
 Wire Wire Line
-	7500 4100 7700 4100
+	6750 4100 6750 4150
 Wire Wire Line
-	7900 4100 7900 4150
+	6350 4450 6350 4500
 Wire Wire Line
-	7700 4050 7700 4100
-Connection ~ 7700 4100
+	6350 4500 6550 4500
 Wire Wire Line
-	7700 4100 7900 4100
+	6750 4500 6750 4450
 Wire Wire Line
-	7500 4450 7500 4500
+	6550 4500 6550 4550
+Connection ~ 6550 4500
 Wire Wire Line
-	7500 4500 7700 4500
-Wire Wire Line
-	7900 4500 7900 4450
-Wire Wire Line
-	7700 4500 7700 4550
-Connection ~ 7700 4500
-Wire Wire Line
-	7700 4500 7900 4500
+	6550 4500 6750 4500
 $Comp
 L power:GND #PWR0103
 U 1 1 5BA44753
-P 7700 4550
-F 0 "#PWR0103" H 7700 4300 50  0001 C CNN
-F 1 "GND" H 7705 4377 50  0000 C CNN
-F 2 "" H 7700 4550 50  0001 C CNN
-F 3 "" H 7700 4550 50  0001 C CNN
-	1    7700 4550
+P 6550 4550
+F 0 "#PWR0103" H 6550 4300 50  0001 C CNN
+F 1 "GND" H 6555 4377 50  0000 C CNN
+F 2 "" H 6550 4550 50  0001 C CNN
+F 3 "" H 6550 4550 50  0001 C CNN
+	1    6550 4550
 	1    0    0    -1
 $EndComp
@@
 	7700 3000 7500 3000
 Text Label 7500 3000 0    50   ~ 0
-VBUS
+VUSB
 Wire Wire Line
 	7200 3550 6850 3550
@@
 	5600 3150 5900 3150
 Text HLabel 4450 3100 0    50   Input ~ 0
-VBUS
+VUSB
 Text HLabel 4450 3200 0    50   Input ~ 0
 USB_DP
@@
 	4450 3100 4750 3100
 Text Label 4750 3100 2    50   ~ 0
-VBUS
+VUSB
 Text Label 4750 3200 2    50   ~ 0
 USB_DP
@@
 Text Label 5900 3550 2    50   ~ 0
 ID
+Wire Wire Line
+	5600 3550 6000 3550
+Wire Wire Line
+	6350 4100 6750 4100
+Wire Wire Line
+	6750 4100 7700 4100
+Connection ~ 6750 4100
+Wire Wire Line
+	6350 4100 5200 4100
+Connection ~ 6350 4100
+Wire Wire Line
+	5200 3750 5200 4100
+Wire Wire Line
+	5300 3750 5300 3850
+Wire Wire Line
+	7700 4100 7700 4050
+Text Label 6450 4100 0    50   ~ 0
+SHIELD
 $Comp
-L Device:D_Schottky D3
-U 1 1 5BB753F5
+L Device:R R4
+U 1 1 5D1D507C
 P 6150 3550
-F 0 "D3" H 6150 3766 50  0000 C CNN
-F 1 "D_Schottky" H 6150 3675 50  0000 C CNN
-F 2 "Diode_SMD:D_SOD-523" H 6150 3550 50  0001 C CNN
+F 0 "R4" H 6220 3596 50  0000 L CNN
+F 1 "330" H 6220 3505 50  0000 L CNN
+F 2 "Resistor_SMD:R_0603_1608Metric" V 6080 3550 50  0001 C CNN
 F 3 "~" H 6150 3550 50  0001 C CNN
 	1    6150 3550
-	1    0    0    -1
+	0    1    1    0
 $EndComp
-Wire Wire Line
-	5600 3550 6000 3550
 $EndSCHEMATC

Commit message: Started the new design of the PCB's layout.
Parts:
- D1: footprint Package_TO_SOT_SMD:SOT-143_Handsoldering -> Package_TO_SOT_SMD:SOT-143
- R3, R4: footprint Resistor_SMD:R_0603_1608Metric -> Resistor_SMD:R_0603_1608Metric_Pad1.05x0.95mm_HandSolder
Changed lines of the file:
@@
 F 0 "D1" H 7850 3900 50  0000 L CNN
 F 1 "PRTR5V0U2X" H 7850 3200 50  0000 L CNN
-F 2 "Package_TO_SOT_SMD:SOT-143_Handsoldering" H 7760 3550 50  0001 C CNN
+F 2 "Package_TO_SOT_SMD:SOT-143" H 7760 3550 50  0001 C CNN
 F 3 "https://assets.nexperia.com/documents/data-sheet/PRTR5V0U2X.pdf" H 7760 3550 50  0001 C CNN
 	1    7700 3550
@@
 F 0 "R3" H 6820 4346 50  0000 L CNN
 F 1 "1M" H 6820 4255 50  0000 L CNN
-F 2 "Resistor_SMD:R_0603_1608Metric" V 6680 4300 50  0001 C CNN
+F 2 "Resistor_SMD:R_0603_1608Metric_Pad1.05x0.95mm_HandSolder" V 6680 4300 50  0001 C CNN
 F 3 "~" H 6750 4300 50  0001 C CNN
 	1    6750 4300
@@
 F 0 "R4" H 6220 3596 50  0000 L CNN
 F 1 "330" H 6220 3505 50  0000 L CNN
-F 2 "Resistor_SMD:R_0603_1608Metric" V 6080 3550 50  0001 C CNN
+F 2 "Resistor_SMD:R_0603_1608Metric_Pad1.05x0.95mm_HandSolder" V 6080 3550 50  0001 C CNN
 F 3 "~" H 6150 3550 50  0001 C CNN
 	1    6150 3550
