File: hw/PCB/Femtosat.kicad_sch (KiCad schematic)
At the start: 5 parts, among them U4 TRH-G2, U7 SAMD21E, Y1 32.768kHz

Commit message: Modified the design of the femto-satellite. Now it is smaller an it has a temperature sensor to calibrate the magnetometer.
Parts:
- added D2: LED, LED_SMD:LED_0805_2012Metric_Pad1.15x1.40mm_HandSolder, symbol Device:LED
- added R5: 330, Resistor_SMD:R_0603_1608Metric_Pad1.05x0.95mm_HandSolder, symbol Device:R
Connections:
- net DL_CD is gone; now on net TRX_IRQ: U7.7 (PA06/8)
- net GND: now also D2.1 (K)
- net DL_NSS renamed STS_LED
- net STS_LED: now also R5.1
- net MAG_SS renamed T_ALERT
- new net: D2.2 (A), R5.2
Other:
- removed sheet Data logger
- sheet Sensors ports: added ALERT, SCL, SDA; removed MISO, MOSI, SCK, SSN
